File: Eagle/converter adapter - Copy.brd (EAGLE design)
At the start: 93 x 43.5 mm, 28 parts

Commit message: adc, leds init
Parts:
- removed IN3, OUT3: (no value), con-ptr500:AK500/2-H
- removed JP7, JP8, VIN3, VOUT3: (no value), pinhead:1X01
- removed U$4: (no value), synergia_logo:SYNERGIA_12MM
- added LED1, LED2, LED3, LED4, LED5, LED6: (no value), led:LED3MM
- added R1, R2, R3, R4, R5, R6: (no value), resistor:R0805
- added SV1, SV10, SV2, SV3, SV6, SV8: (no value), con-lstb:MA04-1
- added SV5, SV7, SV9: (no value), con-harting-ml:ML10
- added U1, U2, U3: HC_05, SerialPortBluetooth:BLUETOOTH_SMD
- moved OUT2 7.04 mm to (67.0, 4.26)
- moved IN2 7.02 mm to (64.0, 38.9)
- moved JP5 7.02 mm to (70.9, 30.4)
- moved JP6 7.02 mm to (70.8, 12.2)
- moved VIN2 7.02 mm to (60.1, 30.4)
- moved VOUT2 7.02 mm to (60.1, 12.1)
- moved U$3 7.00 mm to (57.0, 16.0)
- moved OUT1 3.09 mm to (39.0, 4.26)
- moved IN1 3.04 mm to (36.0, 38.9)
- moved JP1 3.04 mm to (42.9, 30.4)
- moved JP3 3.04 mm to (42.8, 12.2)
- moved VIN1 3.04 mm to (32.1, 30.4)
- moved VOUT1 3.04 mm to (32.1, 12.1)
- moved U$2 3.00 mm to (29.0, 16.0)
- moved OUT 0.75 mm to (12.0, 4.26)
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Connections:
- removed net GND3: IN3.2, JP7.1, JP8.1, OUT3.1
- removed net N$13: OUT3.2, VOUT3.1
- removed net N$14: IN3.1, VIN3.1
- new net +3V1: SV5.2, U1.12
- new net +3V2: SV7.2, U2.12
- new net +3V3: SV9.2, U3.12
- new net GND4: R1.2, R2.2, SV5.1, U1.13, U1.21, U1.22
- new net GND5: R3.2, R4.2, SV7.1, U2.13, U2.21, U2.22
- new net GND6: R5.2, R6.2, SV9.1, U3.13, U3.21, U3.22
- new net N$17: SV5.5, U1.1
- new net N$18: SV5.6, U1.2
- new net N$19: LED2.A, U1.31
- new net N$20: LED1.A, U1.32
- new net N$21: LED1.K, R1.1
- new net N$22: LED2.K, R2.1
- new net N$23: SV7.5, U2.1
- new net N$24: SV7.6, U2.2
- new net N$25: LED4.A, U2.31
- new net N$26: LED3.A, U2.32
- new net N$27: LED3.K, R3.1
- new net N$28: LED4.K, R4.1
- new net N$29: SV9.5, U3.1
- new net N$30: SV9.6, U3.2
- new net N$31: LED6.A, U3.31
- new net N$32: LED5.A, U3.32
- new net N$33: LED5.K, R5.1
- new net N$34: LED6.K, R6.1
Routing:
- net GND6: track 0.00 -> 67.3 mm
- net GND5: track 0.00 -> 67.3 mm
- net GND4: track 0.00 -> 67.3 mm
- net +3V3: track 0.00 -> 59.8 mm
- net +3V1: track 0.00 -> 59.8 mm
- net +3V2: track 0.00 -> 59.8 mm
- net N$24: track 0.00 -> 36.0 mm
- net N$18: track 0.00 -> 36.0 mm
- net N$30: track 0.00 -> 36.0 mm
- net N$29: track 0.00 -> 17.1 mm
- net N$23: track 0.00 -> 17.1 mm
- net N$17: track 0.00 -> 17.1 mm
- net N$32: track 0.00 -> 7.51 mm
- net N$26: track 0.00 -> 7.51 mm
- net N$20: track 0.00 -> 7.51 mm
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- added copper zone on layer 16, net GND4
- added copper zone on layer 16, net GND5
- added copper zone on layer 16, net GND6
- removed copper zone on layer 16, net GND3
- removed copper zone on layer 16, net N$13
- removed copper zone on layer 16, net N$14
- removed copper zone on layer 16, net N$15
- removed copper zone on layer 16, net N$16
Other:
- board size 93 x 43.5 mm -> 91.1 x 96.6 mm
