File: Eagle/converter adapter.sch (EAGLE design)
At the start: 6 parts

Commit message: adc, leds init
Parts:
- added SV1: (no value), con-lstb:MA04-1
Changed lines of the file:
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@@
 <part name="OUT" library="con-ptr500" deviceset="AK500/2-H" device=""/>
 <part name="GND1" library="supply1" deviceset="GND" device=""/>
+<part name="SV1" library="con-lstb" deviceset="MA04-1" device=""/>
 </parts>
 <sheets>
@@
 <instance part="OUT" gate="-2" x="86.36" y="45.72" rot="R180"/>
 <instance part="GND1" gate="1" x="68.58" y="30.48"/>
+<instance part="SV1" gate="1" x="50.8" y="60.96"/>
 </instances>
 <busses>
